File: pcb/numb12_driver.kicad_sch (KiCad schematic)
At the start: 19 parts, among them Q1 AOD413A(UMW), U5 LM3409MY/NOPB

Commit message: update pcb
Parts:
- added R17: 10k, Resistor_SMD:R_0603_1608Metric, symbol Device:R
- C10, C11, C12, C13, C4, C5, C6, C9: value 4.7uF -> 4.7uF 35V; LCSC Part (none) -> C307467
- C7: value 1uF -> 1uF 50V; LCSC Part (none) -> C5199872
- C8: value 470pF -> 470pF 50V; LCSC Part (none) -> C16194503
Connections:
- net GND: now also R17.2
- net PWM: now also R17.1

Commit message: finalize bom
Parts:
- R1: LCSC Part (none) -> C861451
- R17: LCSC Part (none) -> C2906982
- R2: LCSC Part (none) -> C2907055
- R4: LCSC Part (none) -> C723488
- R5: LCSC Part (none) -> C2904225
Changed lines of the file:
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@@
+			)
+		)
+		(property "LCSC Part" "C2907055"
+			(at 54.61 69.85 0)
+			(hide yes)
+			(show_name no)
+			(do_not_autoplace no)
+			(effects
+				(font
+					(size 1.27 1.27)
+				)
 			)
 		)
@@
 			)
 		)
+		(property "LCSC Part" "C2906982"
+			(at 162.56 76.2 0)
+			(hide yes)
+			(show_name no)
+			(do_not_autoplace no)
+			(effects
+				(font
+					(size 1.27 1.27)
+				)
+			)
+		)
 		(pin "1"
 		)
@@
 			)
 		)
+		(property "LCSC Part" "C723488"
+			(at 77.47 77.47 0)
+			(hide yes)
+			(show_name no)
+			(do_not_autoplace no)
+			(effects
+				(font
+					(size 1.27 1.27)
+				)
+			)
+		)
 		(pin "2"
 		)
@@
 			)
 		)
+		(property "LCSC Part" "C2904225"
+			(at 124.46 74.93 0)
+			(hide yes)
+			(show_name no)
+			(do_not_autoplace no)
+			(effects
+				(font
+					(size 1.27 1.27)
+				)
+			)
+		)
 		(pin "2"
 		)
@@
 			(at 54.61 62.23 0)
 			(hide yes)
+			(show_name no)
+			(do_not_autoplace no)
+			(effects
+				(font
+					(size 1.27 1.27)
+				)
+			)
+		)
+		(property "LCSC Part" "C861451"
+			(at 54.61 62.23 0)
+			(hide yes)
