File: pcb/numb12_driver.kicad_sch (KiCad schematic)
At the start: 20 parts, among them Q1 AOD413A(UMW), U5 LM3409MY/NOPB

Commit message: update board after coil whine mitigations
Parts:
- C10, C11, C12, C9: now not fitted
- L1: value APH1265T220M -> SMPQ1306-220MT; LCSC Part C5349635 -> C22396364
Changed lines of the file:
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@@
 			)
 		)
-		(property "Value" "APH1265T220M"
+		(property "Value" "SMPQ1306-220MT"
 			(at 111.76 89.916 0)
 			(show_name no)
@@
 			)
 		)
-		(property "LCSC Part" "C5349635"
+		(property "LCSC Part" "C22396364"
 			(at 111.76 102.87 0)
 			(hide yes)
@@
 		(on_board yes)
 		(in_pos_files yes)
-		(dnp no)
+		(dnp yes)
 		(property "Reference" "C9"
 			(at 101.346 99.568 0)
@@
 		(on_board yes)
 		(in_pos_files yes)
-		(dnp no)
+		(dnp yes)
 		(property "Reference" "C12"
 			(at 116.586 99.568 0)
@@
 		(on_board yes)
 		(in_pos_files yes)
-		(dnp no)
+		(dnp yes)
 		(property "Reference" "C11"
 			(at 111.506 99.568 0)
@@
 		(on_board yes)
 		(in_pos_files yes)
-		(dnp no)
+		(dnp yes)
 		(property "Reference" "C10"
 			(at 106.426 99.568 0)
