File: pcb/power.kicad_sch (KiCad schematic)
At the start: 17 parts, among them U1 AP63205WU-7, U2 CH224A, U4 AMS1117-3.3

Commit message: finalize bom
Parts:
- R22, R23: LCSC Part (none) -> C2907005
- R24: LCSC Part (none) -> C2907095
Changed lines of the file:
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@@
+			)
+		)
+		(property "LCSC Part" "C2907005"
+			(at 129.54 39.37 0)
+			(hide yes)
+			(show_name no)
+			(do_not_autoplace no)
+			(effects
+				(font
+					(size 1.27 1.27)
+				)
 			)
 		)
@@
 			)
 		)
+		(property "LCSC Part" "C2907005"
+			(at 125.73 39.37 0)
+			(hide yes)
+			(show_name no)
+			(do_not_autoplace no)
+			(effects
+				(font
+					(size 1.27 1.27)
+				)
+			)
+		)
 		(pin "1"
 		)
@@
 			(at 83.82 58.42 0)
 			(hide yes)
+			(show_name no)
+			(do_not_autoplace no)
+			(effects
+				(font
+					(size 1.27 1.27)
+				)
+			)
+		)
+		(property "LCSC Part" "C2907095"
+			(at 83.82 58.42 0)
+			(hide yes)
