File: pcb/truecolors_driver.kicad_pcb (KiCad board)
At the start: 4 copper layers, 70 x 90 mm, 106 parts, among them CN1 1.0-3PWT, CN2 47053-1000, Q1 AOD413A(UMW), Q2 AOD413A(UMW), Q3 AOD413A(UMW), Q4 BSS138, SW1 TS-1088-AR02016, U1 AP63205WU-7, U2 CH224A, U3 ESP32-S3-WROOM-1(N8R8)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

Commit message: add status led
Parts:
- added LED1: WS2812B-B, EasyEDA:LED-SMD_4P-L5.0-W5.0-BL_TC5050RGB, F.Cu at (97.3, 127.3)
- added TP10: 5V, TestPoint:TestPoint_Pad_D2.0mm, F.Cu at (95.0, 132.6)
- added TP11: D, TestPoint:TestPoint_Pad_D2.0mm, F.Cu at (98.0, 132.6)
- added TP9: GND, TestPoint:TestPoint_Pad_D2.0mm, F.Cu at (101.0, 132.5)
Connections:
- H1 pad 1: unconnected-(H1-Pad1) -> GND
- H2 pad 1: unconnected-(H2-Pad1) -> GND
- H3 pad 1: unconnected-(H3-Pad1) -> GND
- H4 pad 1: unconnected-(H4-Pad1) -> GND
- H5 pad 1: unconnected-(H5-Pad1) -> GND
- U3 pad 19: unconnected-(U3-IO11-Pad19) -> /LED_DIN
Routing:
- net /LED_DIN: track 0.00 -> 9.52 mm
- net +5V: track 50.8 -> 54.7 mm, vias 8 -> 9
- net Net-(LED1-DOUT): track 0.00 -> 3.18 mm
- net GND: vias 39 -> 49
