File: pcb/truecolors_driver.kicad_pcb (KiCad board)
At the start: 4 copper layers, 70 x 90 mm, 110 parts, among them CN1 1.0-3PWT, CN2 47053-1000, Q1 AOD413A(UMW), Q2 AOD413A(UMW), Q3 AOD413A(UMW), Q4 BSS138, SW1 TS-1088-AR02016, U1 AP63205WU-7, U2 CH224A, U3 ESP32-S3-WROOM-1(N8R8)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

Commit message: fix typo
Other:
- board text added: "CAUTION - CLASS 4 LASER RADIATION WHEN DISASSEMBLED"
- board text removed: "CAUTION - CLASS 4 LASER RADIATION WHEN DISASSEMBLED AND DIFFUSOR OPTICS REMOVED"
Changed lines of the file:
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@@
 		)
 	)
-	(gr_text "CAUTION - CLASS 4 LASER\nRADIATION WHEN DISASSEMBLED\nAND DIFFUSOR OPTICS REMOVED"
+	(gr_text "CAUTION - CLASS 4 LASER\nRADIATION WHEN DISASSEMBLED"
 		(at 110 109 0)
 		(layer "F.SilkS" knockout)
@@
 	)
 	(zone
+		(net "/D+")
+		(layer "F.Cu")
+		(hatch none 0.1)
+		(priority 30001)
+		(attr
+			(teardrop
+				(type padvia)
+			)
+		)
+		(connect_pads yes
+			(clearance 0)
+		)
+		(min_thickness 0.0254)
+		(fill yes
+			(island_removal_mode 1)
+		)
+		(polygon
+			(pts
+				(xy 84.98709 132.04537) (xy 85.212258 132.175366) (xy 85.212258 132.175367) (xy 85.229054 132.123051)
+				(xy 85.585 131.75) (xy 85.207918 131.006143) (xy 84.685 131.75) (xy 84.970294 132.097685) (xy 84.98709 132.045369)
+			)
+		)
+	)
+	(zone
 		(net "GND")
 		(layer "F.Cu")
@@
 			)
 		)
-	)
-	(zone
-		(net "/D+")
-		(layer "F.Cu")
-		(hatch none 0.1)
-		(priority 30001)
-		(attr
-			(teardrop
-				(type padvia)
-			)
-		)
-		(connect_pads yes
-			(clearance 0)
-		)
-		(min_thickness 0.0254)
-		(fill yes
-			(island_removal_mode 1)
-		)
-		(polygon
-			(pts
-				(xy 84.98709 132.04537) (xy 85.212258 132.175366) (xy 85.212258 132.175367) (xy 85.229054 132.123051)
-				(xy 85.585 131.75) (xy 85.207918 131.006143) (xy 84.685 131.75) (xy 84.970294 132.097685) (xy 84.98709 132.045369)
-			)
-		)
