File: pcb/truecolors_driver.kicad_sch (KiCad schematic)
At the start: 9 parts, among them SW1 TS-1088-AR02016, U2 CH224A, U3 ESP32-S3-WROOM-1(N8R8), U4 AMS1117-3.3

Commit message: update pcb
Parts:
- added C34, C36, C37, C38, C39: 10uF 25V, Capacitor_SMD:C_0603_1608Metric, symbol Device:C
- added C35, C40: 100nF 16V, Capacitor_SMD:C_0603_1608Metric, symbol Device:C
- added CN1: 1.0-3PWT, EasyEDA:CONN-SMD_3P-P1.00_C3029342, symbol EasyEDA:1.0-3PWT
- added CN2: 47053-1000, EasyEDA:CONN-TH_47053-1000, symbol EasyEDA:47053-1000
- added L4: 4.7uH, EasyEDA:IND-SMD_L4.4-W4.2, symbol EasyEDA:APH0420T4R7M
- added Q4: BSS138, Package_TO_SOT_SMD:SOT-23, symbol Transistor_FET:BSS138
- added R20, R25: 10k, Resistor_SMD:R_0603_1608Metric, symbol Device:R
- added R21: 68k, Resistor_SMD:R_0603_1608Metric, symbol Device:R
- added R22, R23: 2k2, Resistor_SMD:R_0603_1608Metric, symbol Device:R
- added R24, R26: 120k, Resistor_SMD:R_0603_1608Metric, symbol Device:R
- added U1: AP63205WU-7, EasyEDA:TSOT-23-6_L2.9-W1.6-P0.95-LS2.8-BL, symbol EasyEDA:AP63205WU-7
- C1: value 1uF -> 1uF 50V; footprint Capacitor_SMD:C_0603_1608Metric_Pad1.08x0.95mm_HandSolder -> Capacitor_SMD:C_0603_1608Metric; LCSC Part (none) -> C5199872
- C2, C3: value 10uF -> 10uF 25V; footprint Capacitor_SMD:C_0603_1608Metric_Pad1.08x0.95mm_HandSolder -> Capacitor_SMD:C_0603_1608Metric; LCSC Part (none) -> C96446
Connections:
- net +20V: now also C34.1, R21.1, U1.2 (EN), U1.3 (VIN)
- net +3.3V: now also R22.1, R23.1, R25.1
- net +5V: now also C36.1, C37.1, C38.1, C39.1, CN2.2, L4.2, U1.1 (FB)
- net GND: now also C34.2, C36.2, C37.2, C38.2, C39.2, C40.1, CN1.2, CN1.4, CN1.5, CN2.1, Q4.2 (S), R20.2, R24.2, R26.2, U1.4 (GND); no longer U2.9 (CFG1)
- net RX: now also CN1.1
- net TX: now also CN1.3
- net CH224A_SDA: now reaches U3.12 (IO8)
- net CH224A_SDA: now also U2.3 (CFG3/SDA), R22.2
- net CH224A_SCL: now reaches U3.17 (IO9)
- net CH224A_SCL: now also U2.2 (CFG2/SCL), R23.2
- net EN_B: now reaches U3.31 (IO38)
- net EN_G: now reaches U3.32 (IO39)
- net EN_R: now reaches U3.33 (IO40)
- net VIN_ADC: now reaches U3.4 (IO4)
- net VIN_ADC: now also C40.2, R20.1, R21.2
- net FAN_PWM: now reaches U3.6 (IO6)
- net FAN_PWM: now also Q4.1 (G), R26.1
- net FAN_TACH: now reaches U3.7 (IO7)
- net FAN_TACH: now also CN2.3, R25.2
- net PD_PG: no longer names the net of U2.10 (PG)
- new net: C35.2, L4.1, U1.5 (SW)
- new net: C35.1, U1.6 (BST)
- new net: CN2.4, Q4.3 (D)
- new net: R24.1, U2.9 (CFG1)
- no-connect marks 6 -> 5
Other:
- moved on the sheet: C1, C2, C3, R16, SW1, U2, U3, U4, USBC1

Commit message: R26 pullup instead of pulldown for fan-off boot
Connections:
- net +3.3V: now also R26.2
- net GND: no longer R26.2
Other:
- moved on the sheet: R26
Changed lines of the file:
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@@
 	)
 	(junction
-		(at 130.81 85.09)
-		(diameter 0)
-		(color 0 0 0 0)
-	)
-	(junction
 		(at 130.81 106.68)
 		(diameter 0)
@@
 	)
 	(junction
-		(at 123.19 77.47)
+		(at 134.62 120.65)
 		(diameter 0)
 		(color 0 0 0 0)
 	)
 	(junction
-		(at 134.62 120.65)
+		(at 123.19 77.47)
 		(diameter 0)
 		(color 0 0 0 0)
@@
 	(wire
 		(pts
-			(xy 123.19 85.09) (xy 130.81 85.09)
-		)
-		(stroke
-			(width 0)
-			(type default)
-		)
-	)
-	(wire
-		(pts
 			(xy 74.93 40.64) (xy 81.28 40.64)
 		)
@@
 	(wire
 		(pts
+			(xy 123.19 72.39) (xy 123.19 77.47)
+		)
+		(stroke
+			(width 0)
+			(type default)
+		)
+	)
+	(wire
+		(pts
 			(xy 29.21 180.34) (xy 29.21 181.61)
 		)
@@
 	)
 	(symbol
+		(lib_id "power:+3.3V")
+		(at 123.19 64.77 0)
+		(unit 1)
+		(body_style 1)
+		(exclude_from_sim no)
+		(in_bom yes)
+		(on_board yes)
+		(in_pos_files yes)
+		(dnp no)
+		(fields_autoplaced yes)
+		(property "Reference" "#PWR042"
+			(at 123.19 68.58 0)
+			(hide yes)
+			(show_name no)
+			(do_not_autoplace no)
+			(effects
+				(font
+					(size 1.27 1.27)
+				)
+			)
+		)
+		(property "Value" "+3.3V"
+			(at 123.19 59.69 0)
+			(show_name no)
+			(do_not_autoplace no)
+			(effects
+				(font
+					(size 1.27 1.27)
+				)
+			)
+		)
+		(property "Footprint" ""
+			(at 123.19 64.77 0)
+			(hide yes)
+			(show_name no)
+			(do_not_autoplace no)
+			(effects
+				(font
+					(size 1.27 1.27)
+				)
+			)
+		)
+		(property "Datasheet" ""
+			(at 123.19 64.77 0)
+			(hide yes)
+			(show_name no)
+			(do_not_autoplace no)
+			(effects
+				(font
+					(size 1.27 1.27)
+				)
+			)
+		)
+		(property "Description" "Power symbol creates a global label with name \"+3.3V\""
+			(at 123.19 64.77 0)
+			(hide yes)
+			(show_name no)
+			(do_not_autoplace no)
+			(effects
+				(font
+					(size 1.27 1.27)
+				)
+			)
+		)
+		(pin "1"
+		)
+		(instances
+			(project "truecolors_driver"
+				(path "/5ee6f65d-ffa4-4e70-aae0-693484c61116"
+					(reference "#PWR042")
+					(unit 1)
+				)
+			)
+		)
+	)
+	(symbol
 		(lib_id "power:+15V")
 		(at 259.08 130.81 0)
@@
 	(symbol
 		(lib_id "Device:R")
-		(at 123.19 81.28 0)
+		(at 123.19 68.58 180)
 		(unit 1)
 		(body_style 1)
@@
 		(dnp no)
 		(property "Reference" "R26"
-			(at 116.332 80.0099 0)
+			(at 130.048 69.8501 0)
 			(show_name no)
 			(do_not_autoplace no)
@@
 		)
 		(property "Value" "120k"
-			(at 116.332 82.5499 0)
+			(at 130.048 67.3101 0)
 			(show_name no)
 			(do_not_autoplace no)
@@
 		)
 		(property "Footprint" "Resistor_SMD:R_0603_1608Metric"
-			(at 121.412 81.28 90)
+			(at 124.968 68.58 90)
 			(hide yes)
 			(show_name no)
@@
 		)
 		(property "Datasheet" ""
-			(at 123.19 81.28 0)
+			(at 123.19 68.58 0)
 			(hide yes)
 			(show_name no)
@@
 		)
 		(property "Description" "Resistor"
-			(at 123.19 81.28 0)
+			(at 123.19 68.58 0)
 			(hide yes)
 			(show_name no)
@@
 		(dnp no)
 		(property "Reference" "Q4"
-			(at 119.888 70.6119 0)
+			(at 114.554 70.6119 0)
 			(show_name no)
 			(do_not_autoplace no)
@@
 		)
 		(property "Value" "BSS138"
-			(at 119.888 73.1519 0)
+			(at 114.554 73.1519 0)
 			(show_name no)
 			(do_not_autoplace no)

Commit message: add mic, add ntc, fix all drc errors
Parts:
- added C41, C43: 100nF 16V, Capacitor_SMD:C_0603_1608Metric, symbol Device:C
- added C42: 10uF 25V, Capacitor_SMD:C_0603_1608Metric, symbol Device:C
- added MIC1: MSM261DGT003, EasyEDA:MIC-SMD_6P-L4.0-W2.0_LMD4020T261-OC3, symbol EasyEDA:MSM261DGT003
- added R27: 10k, Resistor_SMD:R_0603_1608Metric, symbol Device:R
- added TP1: NTC+, TestPoint:TestPoint_Keystone_5019_Miniature, symbol Connector:TestPoint
- added TP2: NTC-, TestPoint:TestPoint_Keystone_5019_Miniature, symbol Connector:TestPoint
Connections:
- net +3.3V: now also C41.2, C42.1, MIC1.1 (VDD), R27.1
- net GND: now also C41.1, C42.2, C43.1, MIC1.2 (GND), MIC1.5 (GND), MIC1.6 (L/R), TP2.1
- net BOOT: now reaches R16.2, SW1.2, U3.27 (IO0)
- net NTC_ADC: now reaches U3.18 (IO10)
- net NTC_ADC: now also C43.2, R27.2, TP1.1
- net MIC_CLK: now reaches U3.20 (IO12)
- net MIC_CLK: now also MIC1.4 (CLK)
- net MIC_DATA: now reaches U3.21 (IO13)
- net MIC_DATA: now also MIC1.3 (DATA)
Other:
- moved on the sheet: C40, CN1, R16, R20, R21, SW1, U3

Commit message: refactor schematic
Parts:
- removed C1: 1uF 50V, Capacitor_SMD:C_0603_1608Metric, symbol Device:C
- removed C2, C3, C34, C36, C37, C38, C39: 10uF 25V, Capacitor_SMD:C_0603_1608Metric, symbol Device:C
- removed C35: 100nF 16V, Capacitor_SMD:C_0603_1608Metric, symbol Device:C
- removed L4: 4.7uH, EasyEDA:IND-SMD_L4.4-W4.2, symbol EasyEDA:APH0420T4R7M
- removed R22, R23: 2k2, Resistor_SMD:R_0603_1608Metric, symbol Device:R
- removed R24: 120k, Resistor_SMD:R_0603_1608Metric, symbol Device:R
- removed U1: AP63205WU-7, EasyEDA:TSOT-23-6_L2.9-W1.6-P0.95-LS2.8-BL, symbol EasyEDA:AP63205WU-7
- removed U2: CH224A, easyeda2kicad:ESSOP-10_L4.9-W3.9-P1.0-LS6.0-TL-EP, symbol easyeda2kicad:CH224A
- removed U4: AMS1117-3.3, easyeda2kicad:SOT-223-3_L6.5-W3.4-P2.30-LS7.0-BR, symbol easyeda2kicad:AMS1117-3.3
- removed USBC1: TYPE-C-31-M-12, easyeda2kicad:USB-C_SMD-TYPE-C-31-M-12_1, symbol easyeda2kicad:TYPE-C-31-M-12
- added TP3: R+, TestPoint:TestPoint_Keystone_5019_Miniature, symbol Connector:TestPoint
- added TP4, TP6, TP8: GND, TestPoint:TestPoint_Keystone_5019_Miniature, symbol Connector:TestPoint
- added TP5: G+, TestPoint:TestPoint_Keystone_5019_Miniature, symbol Connector:TestPoint
- added TP7: B+, TestPoint:TestPoint_Keystone_5019_Miniature, symbol Connector:TestPoint
Connections:
- net GND: now also TP4.1, TP6.1, TP8.1
- net driverB/VOUT: now also TP7.1
- net driverG/VOUT: now also TP5.1
- net driverR/VOUT: now also TP3.1
- no-connect marks 5 -> 20
Other:
- added sheet power (power.kicad_sch)
- moved on the sheet: C40, C41, C42, C43, CN1, CN2, MIC1, Q4, R20, R21, R25, R26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

Commit message: add mounting holes, labels
Parts:
- added H1, H2, H3, H4, H5: M3, MountingHole:MountingHole_3.2mm_M3_DIN965_Pad, symbol Mechanical:MountingHole

Commit message: finalize bom
Parts:
- H1, H2, H3, H4, H5: symbol Mechanical:MountingHole -> Mechanical:MountingHole_Pad
- R16, R20, R25, R27: LCSC Part (none) -> C2906982
- R21: LCSC Part (none) -> C114633
- R26: LCSC Part (none) -> C2907095
- TP1, TP2, TP3, TP4, TP5, TP6, TP7, TP8: now left out of the parts list
Connections:
- no-connect marks 20 -> 25
Changed lines of the file:
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@@
 	)
 	(no_connect
+		(at 26.67 71.12)
+	)
+	(no_connect
 		(at 160.02 109.22)
 	)
 	(no_connect
+		(at 34.29 71.12)
+	)
+	(no_connect
 		(at 160.02 81.28)
 	)
@@
 	)
 	(no_connect
+		(at 41.91 71.12)
+	)
+	(no_connect
 		(at 160.02 91.44)
 	)
 	(no_connect
+		(at 49.53 71.12)
+	)
+	(no_connect
 		(at 143.51 124.46)
 	)
 	(no_connect
+		(at 19.05 71.12)
+	)
+	(no_connect
 		(at 151.13 124.46)
 	)
@@
 		(body_style 1)
 		(exclude_from_sim no)
-		(in_bom yes)
+		(in_bom no)
 		(on_board yes)
 		(in_pos_files yes)
@@
 	)
 	(symbol
-		(lib_id "Mechanical:MountingHole")
-		(at 24.13 80.01 0)
+		(lib_id "Mechanical:MountingHole_Pad")
+		(at 34.29 68.58 0)
 		(unit 1)
 		(body_style 1)
@@
 		(fields_autoplaced yes)
 		(property "Reference" "H3"
-			(at 26.67 78.7399 0)
+			(at 36.83 66.0399 0)
 			(show_name no)
 			(do_not_autoplace no)
@@
 		)
 		(property "Value" "M3"
-			(at 26.67 81.2799 0)
+			(at 36.83 68.5799 0)
 			(show_name no)
 			(do_not_autoplace no)
@@
 		)
 		(property "Footprint" "MountingHole:MountingHole_3.2mm_M3_DIN965_Pad"
-			(at 24.13 80.01 0)
+			(at 34.29 68.58 0)
 			(hide yes)
 			(show_name no)
@@
 		)
 		(property "Datasheet" ""
-			(at 24.13 80.01 0)
+			(at 34.29 68.58 0)
 			(hide yes)
 			(show_name no)
@@
 			)
 		)
-		(property "Description" "Mounting Hole"
-			(at 24.13 80.01 0)
+		(property "Description" "Mounting Hole with connection"
+			(at 34.29 68.58 0)
 			(hide yes)
 			(show_name no)
@@
 			)
 		)
+		(pin "1"
+		)
 		(instances
 			(project "truecolors_driver"
@@
 	)
 	(symbol
-		(lib_id "Mechanical:MountingHole")
-		(at 24.13 90.17 0)
+		(lib_id "Mechanical:MountingHole_Pad")
+		(at 49.53 68.58 0)
 		(unit 1)
 		(body_style 1)
@@
 		(fields_autoplaced yes)
 		(property "Reference" "H5"
-			(at 26.67 88.8999 0)
+			(at 52.07 66.0399 0)
 			(show_name no)
 			(do_not_autoplace no)
@@
 		)
 		(property "Value" "M3"
-			(at 26.67 91.4399 0)
+			(at 52.07 68.5799 0)
 			(show_name no)
 			(do_not_autoplace no)
@@
 		)
 		(property "Footprint" "MountingHole:MountingHole_3.2mm_M3_DIN965_Pad"
-			(at 24.13 90.17 0)
+			(at 49.53 68.58 0)
 			(hide yes)
 			(show_name no)
@@
 		)
 		(property "Datasheet" ""
-			(at 24.13 90.17 0)
+			(at 49.53 68.58 0)
 			(hide yes)
 			(show_name no)
@@
 			)
 		)
-		(property "Description" "Mounting Hole"
-			(at 24.13 90.17 0)
+		(property "Description" "Mounting Hole with connection"
+			(at 49.53 68.58 0)
 			(hide yes)
 			(show_name no)
@@
 			)
 		)
+		(pin "1"
+		)
 		(instances
 			(project "truecolors_driver"
@@
 		(body_style 1)
 		(exclude_from_sim no)
-		(in_bom yes)
+		(in_bom no)
 		(on_board yes)
 		(in_pos_files yes)
@@
 		(body_style 1)
 		(exclude_from_sim no)
-		(in_bom yes)
+		(in_bom no)
 		(on_board yes)
 		(in_pos_files yes)
@@
 			)
 		)
+		(property "LCSC Part" "C2906982"
+			(at 149.86 27.94 0)
+			(hide yes)
+			(show_name no)
+			(do_not_autoplace no)
+			(effects
+				(font
+					(size 1.27 1.27)
+				)
+			)
+		)
 		(pin "1"
 		)
@@
 	)
 	(symbol
-		(lib_id "Mechanical:MountingHole")
-		(at 24.13 74.93 0)
+		(lib_id "Mechanical:MountingHole_Pad")
+		(at 26.67 68.58 0)
 		(unit 1)
 		(body_style 1)
@@
 		(fields_autoplaced yes)
 		(property "Reference" "H2"
-			(at 26.67 73.6599 0)
+			(at 29.21 66.0399 0)
 			(show_name no)
 			(do_not_autoplace no)
@@
 		)
 		(property "Value" "M3"
-			(at 26.67 76.1999 0)
+			(at 29.21 68.5799 0)
 			(show_name no)
 			(do_not_autoplace no)
@@
 		)
 		(property "Footprint" "MountingHole:MountingHole_3.2mm_M3_DIN965_Pad"
-			(at 24.13 74.93 0)
+			(at 26.67 68.58 0)
 			(hide yes)
 			(show_name no)
@@
 		)
 		(property "Datasheet" ""
-			(at 24.13 74.93 0)
+			(at 26.67 68.58 0)
 			(hide yes)
 			(show_name no)
@@
 			)
 		)
-		(property "Description" "Mounting Hole"
-			(at 24.13 74.93 0)
+		(property "Description" "Mounting Hole with connection"
+			(at 26.67 68.58 0)
 			(hide yes)
 			(show_name no)
@@
 			)
 		)
+		(pin "1"
+		)
 		(instances
 			(project "truecolors_driver"
@@
 		(body_style 1)
 		(exclude_from_sim no)
-		(in_bom yes)
+		(in_bom no)
 		(on_board yes)
 		(in_pos_files yes)
@@
 			)
 		)
+		(property "LCSC Part" "C2906982"
+			(at 252.73 41.91 0)
+			(hide yes)
+			(show_name no)
+			(do_not_autoplace no)
+			(effects
+				(font
+					(size 1.27 1.27)
+				)
+			)
+		)
 		(pin "1"
 		)
@@
 		(body_style 1)
 		(exclude_from_sim no)
-		(in_bom yes)
+		(in_bom no)
 		(on_board yes)
 		(in_pos_files yes)
@@
 			)
 		)
+		(property "LCSC Part" "C114633"
+			(at 252.73 34.29 0)
+			(hide yes)
+			(show_name no)
+			(do_not_autoplace no)
+			(effects
+				(font
+					(size 1.27 1.27)
+				)
+			)
+		)
 		(pin "1"
 		)
@@
 	)
 	(symbol
-		(lib_id "Mechanical:MountingHole")
-		(at 24.13 85.09 0)
+		(lib_id "Mechanical:MountingHole_Pad")
+		(at 41.91 68.58 0)
 		(unit 1)
 		(body_style 1)
@@
 		(fields_autoplaced yes)
 		(property "Reference" "H4"
-			(at 26.67 83.8199 0)
+			(at 44.45 66.0399 0)
 			(show_name no)
 			(do_not_autoplace no)
@@
 		)
 		(property "Value" "M3"
-			(at 26.67 86.3599 0)
+			(at 44.45 68.5799 0)
 			(show_name no)
 			(do_not_autoplace no)
@@
 		)
 		(property "Footprint" "MountingHole:MountingHole_3.2mm_M3_DIN965_Pad"
-			(at 24.13 85.09 0)
+			(at 41.91 68.58 0)
 			(hide yes)
 			(show_name no)
@@
 		)
 		(property "Datasheet" ""
-			(at 24.13 85.09 0)
+			(at 41.91 68.58 0)
 			(hide yes)
 			(show_name no)
@@
 			)
 		)
-		(property "Description" "Mounting Hole"
-			(at 24.13 85.09 0)
+		(property "Description" "Mounting Hole with connection"
+			(at 41.91 68.58 0)
 			(hide yes)
 			(show_name no)
@@
 			)
 		)
+		(pin "1"
+		)
 		(instances
 			(project "truecolors_driver"
@@
 			)
 		)
+		(property "LCSC Part" "C2906982"
+			(at 255.27 82.55 0)
+			(hide yes)
+			(show_name no)
+			(do_not_autoplace no)
+			(effects
+				(font
+					(size 1.27 1.27)
+				)
+			)
+		)
 		(pin "1"
 		)
@@
 		(body_style 1)
 		(exclude_from_sim no)
-		(in_bom yes)
+		(in_bom no)
 		(on_board yes)
 		(in_pos_files yes)
@@
 			)
 		)
+		(property "LCSC Part" "C2907095"
+			(at 218.44 82.55 0)
+			(hide yes)
+			(show_name no)
+			(do_not_autoplace no)
+			(effects
+				(font
+					(size 1.27 1.27)
+				)
+			)
+		)
 		(pin "1"
 		)
@@
 	)
 	(symbol
-		(lib_id "Mechanical:MountingHole")
-		(at 24.13 69.85 0)
+		(lib_id "Mechanical:MountingHole_Pad")
+		(at 19.05 68.58 0)
 		(unit 1)
 		(body_style 1)
@@
 		(fields_autoplaced yes)
 		(property "Reference" "H1"
-			(at 26.67 68.5799 0)
+			(at 21.59 66.0399 0)
 			(show_name no)
 			(do_not_autoplace no)
@@
 		)
 		(property "Value" "M3"
-			(at 26.67 71.1199 0)
+			(at 21.59 68.5799 0)
 			(show_name no)
 			(do_not_autoplace no)
@@
 		)
 		(property "Footprint" "MountingHole:MountingHole_3.2mm_M3_DIN965_Pad"
-			(at 24.13 69.85 0)
+			(at 19.05 68.58 0)
 			(hide yes)
 			(show_name no)
@@
 		)
 		(property "Datasheet" ""
-			(at 24.13 69.85 0)
+			(at 19.05 68.58 0)
 			(hide yes)
 			(show_name no)
@@
 			)
 		)
-		(property "Description" "Mounting Hole"
-			(at 24.13 69.85 0)
+		(property "Description" "Mounting Hole with connection"
+			(at 19.05 68.58 0)
 			(hide yes)
 			(show_name no)
@@
 			)
 		)
+		(pin "1"
+		)
 		(instances
 			(project "truecolors_driver"
@@
 		(body_style 1)
 		(exclude_from_sim no)
-		(in_bom yes)
+		(in_bom no)
 		(on_board yes)
 		(in_pos_files yes)
@@
 		(body_style 1)
 		(exclude_from_sim no)
-		(in_bom yes)
+		(in_bom no)
 		(on_board yes)
 		(in_pos_files yes)
@@
 			(at 201.93 33.02 0)
 			(hide yes)
+			(show_name no)
+			(do_not_autoplace no)
+			(effects
+				(font
+					(size 1.27 1.27)
+				)
+			)
+		)
+		(property "LCSC Part" "C2906982"
+			(at 201.93 33.02 0)
+			(hide yes)

Commit message: add status led
Parts:
- added LED1: WS2812B-B, EasyEDA:LED-SMD_4P-L5.0-W5.0-BL_TC5050RGB, symbol EasyEDA:WS2812B-B
- added TP10: 5V, TestPoint:TestPoint_Pad_D2.0mm, symbol Connector:TestPoint
- added TP11: D, TestPoint:TestPoint_Pad_D2.0mm, symbol Connector:TestPoint
- added TP9: GND, TestPoint:TestPoint_Pad_D2.0mm, symbol Connector:TestPoint
Connections:
- net +5V: now also LED1.1 (VDD), TP10.1
- net GND: now also H1.1, H2.1, H3.1, H4.1, H5.1, LED1.3 (VSS), TP9.1
- net LED_DIN: now reaches U3.19 (IO11)
- net LED_DIN: now also LED1.4 (DIN)
- new net: LED1.2 (DOUT), TP11.1
- no-connect marks 25 -> 19
